Commit message: Update arm_2026 to work with full pipeline [IN PROGRESS]

File: install/arm_2026/share/arm_2026/description/arm_2026.urdf.xacro (robot description, xacro)
@@ -33,4 +33,20 @@
     </visual>
   </link>
+  <link name="wrist_roll_link">
+    <visual>
+      <origin xyz="0.08 0 0" rpy="0 0 0"/>
+      <geometry>
+        <cylinder radius="0.02" length="0.16"/>
+      </geometry>
+    </visual>
+  </link>
+  <link name="wrist_twist_link">
+    <visual>
+      <origin xyz="0.06 0 0" rpy="0 0 0"/>
+      <geometry>
+        <box size="0.12 0.025 0.025"/>
+      </geometry>
+    </visual>
+  </link>
   <joint name="base_yaw" type="revolute">
     <parent link="base_link"/>
@@ -54,4 +70,18 @@
     <limit lower="-1.57" upper="1.57" effort="10" velocity="0.2"/>
   </joint>
+  <joint name="wrist_roll" type="revolute">
+    <parent link="elbow_link"/>
+    <child link="wrist_roll_link"/>
+    <origin xyz="0.20 0 0" rpy="0 0 0"/>
+    <axis xyz="1 0 0"/>
+    <limit lower="-1.57" upper="1.57" effort="10" velocity="0.5"/>
+  </joint>
+  <joint name="wrist_twist" type="revolute">
+    <parent link="wrist_roll_link"/>
+    <child link="wrist_twist_link"/>
+    <origin xyz="0.16 0 0" rpy="0 0 0"/>
+    <axis xyz="0 0 1"/>
+    <limit lower="-1.57" upper="1.57" effort="10" velocity="0.5"/>
+  </joint>
   <ros2_control name="Arm2026Hardware" type="system">
     <hardware>
@@ -70,4 +100,12 @@
       <state_interface name="position"/>
     </joint>
+    <joint name="wrist_roll">
+      <command_interface name="position"/>
+      <state_interface name="position"/>
+    </joint>
+    <joint name="wrist_twist">
+      <command_interface name="position"/>
+      <state_interface name="position"/>
+    </joint>
   </ros2_control>
 </robot>

Commit message: Update arm_2026 (Fix urdf, fix keyboard teleop, add Logitech Extreme 3D joystick teleop

File: install/arm_2026/share/arm_2026/description/arm_2026.urdf.xacro (robot description, xacro)
@@ -33,17 +33,25 @@
     </visual>
   </link>
+  <!-- Main wrist housing -->
   <link name="wrist_roll_link">
     <visual>
-      <origin xyz="0.08 0 0" rpy="0 0 0"/>
+      <origin xyz="0.025 0 0" rpy="0 0 0"/>
       <geometry>
-        <cylinder radius="0.02" length="0.16"/>
+        <box size="0.05 0.06 0.06"/>
+      </geometry>
+    </visual>
+    <visual>
+      <origin xyz="0.025 0 0" rpy="0 1.5708 0"/>
+      <geometry>
+        <cylinder radius="0.018" length="0.05"/>
       </geometry>
     </visual>
   </link>
+  <!-- Front/output wrist piece, attached very closely -->
   <link name="wrist_twist_link">
     <visual>
-      <origin xyz="0.06 0 0" rpy="0 0 0"/>
+      <origin xyz="0.02 0 0" rpy="0 0 0"/>
       <geometry>
-        <box size="0.12 0.025 0.025"/>
+        <box size="0.04 0.045 0.045"/>
       </geometry>
     </visual>
@@ -56,8 +64,9 @@
     <limit lower="-3.14" upper="3.14" effort="10" velocity="1.0"/>
   </joint>
+  <!-- Zero position now starts 45 degrees upward -->
   <joint name="shoulder_extension" type="revolute">
     <parent link="base_link_1"/>
     <child link="shoulder_link"/>
-    <origin xyz="0 0 0.10" rpy="0 0 0"/>
+    <origin xyz="0 0 0.10" rpy="0 -0.785398 0"/>
     <axis xyz="0 1 0"/>
     <limit lower="-1.57" upper="1.57" effort="10" velocity="0.2"/>
@@ -70,16 +79,18 @@
     <limit lower="-1.57" upper="1.57" effort="10" velocity="0.2"/>
   </joint>
+  <!-- Wrist module starts at forearm tip -->
   <joint name="wrist_roll" type="revolute">
     <parent link="elbow_link"/>
     <child link="wrist_roll_link"/>
     <origin xyz="0.20 0 0" rpy="0 0 0"/>
-    <axis xyz="1 0 0"/>
+    <axis xyz="0 1 0"/>
     <limit lower="-1.57" upper="1.57" effort="10" velocity="0.5"/>
   </joint>
+  <!-- Twist joint is almost co-located with wrist housing -->
   <joint name="wrist_twist" type="revolute">
     <parent link="wrist_roll_link"/>
     <child link="wrist_twist_link"/>
-    <origin xyz="0.16 0 0" rpy="0 0 0"/>
-    <axis xyz="0 0 1"/>
+    <origin xyz="0.03 0 0" rpy="0 0 0"/>
+    <axis xyz="1 0 0"/>
     <limit lower="-1.57" upper="1.57" effort="10" velocity="0.5"/>
   </joint>
