Commit message: Update arm_2026(Added claw joint control, added debug mode which allows bypassing joint limits, and polished up system a bit)

File: src/arm_2026/description/arm_2026.urdf.xacro (robot description, xacro)
@@ -48,5 +48,5 @@
     </visual>
   </link>
-  <!-- Front/output wrist piece, attached very closely -->
+  <!-- Front/output wrist piece -->
   <link name="wrist_twist_link">
     <visual>
@@ -54,4 +54,13 @@
       <geometry>
         <box size="0.04 0.045 0.045"/>
+      </geometry>
+    </visual>
+  </link>
+  <!-- Simple claw visual -->
+  <link name="claw_link">
+    <visual>
+      <origin xyz="0.03 0 0" rpy="0 0 0"/>
+      <geometry>
+        <box size="0.06 0.02 0.02"/>
       </geometry>
     </visual>
@@ -95,4 +104,12 @@
     <limit lower="-1.57" upper="1.57" effort="10" velocity="0.5"/>
   </joint>
+  <!-- Claw attached after wrist twist -->
+  <joint name="claw" type="revolute">
+    <parent link="wrist_twist_link"/>
+    <child link="claw_link"/>
+    <origin xyz="0.04 0 0" rpy="0 0 0"/>
+    <axis xyz="0 1 0"/>
+    <limit lower="-1.57" upper="1.57" effort="10" velocity="0.5"/>
+  </joint>
   <ros2_control name="Arm2026Hardware" type="system">
     <hardware>
@@ -119,4 +136,8 @@
       <state_interface name="position"/>
     </joint>
+    <joint name="claw">
+      <command_interface name="position"/>
+      <state_interface name="position"/>
+    </joint>
   </ros2_control>
 </robot>
